File: board/my_project.kicad_sch (KiCad schematic)
At the start: 3 parts, among them U1 LT1762

Commit message: only values changes
Parts:
- R1: value 10k -> 33k
- R2: value 10k -> 9k
Changed lines of the file:
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@@
 			)
 		)
-		(property "Value" "10k"
+		(property "Value" "9k"
 			(at 162.56 100.3299 0)
 			(effects
@@
 			)
 		)
-		(property "Value" "10k"
+		(property "Value" "33k"
 			(at 162.56 92.7099 0)
 			(effects
